File: TG-Watch02B-rev04.sch (EAGLE design)
At the start: 62 parts, among them IC3 W25Q128JVSIQ TR, Q3 DMG2305, U10 MCU-ATTINY10, U2 BQ27441-G1, U4 FAN5331SX, U7 DISP_1.54_LCMTF15423A-C_LCD+C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, U8 UNDERVOLT-TPS3702CX3, U9 MCP73831/OT

Commit message: chagne battery IC and make path for rev02 boards
Parts:
- removed C2, C4: 1uf, 0TG-Lib v01.5:C-US__0402_NOMASK
- removed R1: .01 ohm, 0TG-Lib v01.5:R_TG_0402
- removed U2: BQ27441-G1, battery-management-temp:BQ27441-G1
- added IC1: LC709203F, microbuilder:LC709203F
- added R13: 10k, 0TG-Lib v01.5:R_TG_0402
- added R3: 11k, 0TG-Lib v01.5:R_TG_0402
Connections:
- removed net 1.8V: C4.2, U2.VDD
- removed net A0: MDBT1.P0.04/AIN2
- removed net D12_SMC_RESET: ISP1.RST, MDBT1.P0.08, R15.2, U10./RST
- removed net GPOUT: U2.GPOUT
- removed net TS: U2.BIN
- removed net VBAT_RAW: BAT1.VBAT, C2.2, R1.2, R6.2, U2.BAT, U2.SRP
- new net A0_SMC_RESET: ISP1.RST, MDBT1.P0.04/AIN2, R15.2, U10./RST
- new net D12_BAT_INT: IC1.ALARMB, MDBT1.P0.08, R13.2
- new net TSENSE: IC1.TSENSE, R3.2
- new net TSW: IC1.TSW, R3.1
- net 3V3: now also R13.1
- net GND: now also IC1.TEST, IC1.VSS; no longer C2.1, C4.1, U2.PWPD, U2.VSS
- net SCL: now also IC1.SCL; no longer U2.SCL
- net SDA: now also IC1.SDA; no longer U2.SDA
- net VBAT: now also BAT1.VBAT, IC1.VDD, R6.2; no longer R1.1, U2.SRN
Other:
- note removed: "I2C ADDR: 0x55"
- note removed: "VDD is 1.8V generated internally"
