File: bat-brd-rev02-panel.brd (EAGLE design)
At the start: 15.5 x 12.5 mm, 18 parts

Commit message: pre-order
Routing:
- net S$9: track 0.00 -> 6.74 mm
- net S$8: track 0.00 -> 6.74 mm
- net S$7: track 0.00 -> 6.74 mm
- net S$6: track 0.00 -> 6.74 mm
- net S$5: track 0.00 -> 6.74 mm
- net S$4: track 0.00 -> 6.74 mm
- net S$3: track 0.00 -> 6.74 mm
- net S$2: track 0.00 -> 6.74 mm
- net S$1: track 0.00 -> 6.74 mm
- net S$20: track 0.00 -> 1.71 mm
- net S$19: track 0.00 -> 1.71 mm
- net S$18: track 0.00 -> 1.71 mm
- net S$17: track 0.00 -> 1.71 mm
- net S$16: track 0.00 -> 1.71 mm
- net S$15: track 0.00 -> 1.71 mm
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