File: TG-Watch02B-rev04.brd (EAGLE design)
At the start: 36.8 x 40.6 mm, 66 parts, among them IC3 W25Q128JVSIQ TR, J1 USB-C-CON-TG_MOD-2295018-2.0, J2 DISP_1.54_LCMTF15423A-C_LCD+C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, J3 CON-BAT-TG-MEZ_FEMALE, Q3 DMG2305, U2 MICROBUILDER_LSM6DSOX, U3 VREG-TPS63036, U4 FAN5331SX, U5 MCP73831/OT, U6 LC709203F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

Commit message: 2022jul07
Parts:
- 04.1: value TG-Watch02B -> TG-Watch
- moved R14 0.65 mm to (27.4, 11.2)
- moved C2 0.25 mm to (27.2, 14.8)
- moved R13 0.15 mm to (27.5, 12.8)
- moved C4 0.05 mm to (27.5, 13.8)
- renumbered 04 to 04.1
