File: TG-Watch02B-rev05.brd (EAGLE design)
At the start: 36.8 x 40.6 mm, 66 parts, among them IC3 W25Q128JVSIQ TR, J1 USB-C-CON-TG_MOD-2295018-2.0, J2 DISP_1.54_LCMTF15423A-C_LCD+C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, J3 CON-BAT-TG-MEZ_FEMALE, Q3 DMG2305, U2 MICROBUILDER_LSM6DSOX, U3 VREG-TPS63036, U4 FAN5331SX, U5 MCP73831/OT, U6 LC709203F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

Commit message: 2022jul07
Parts:
- 04.1: value TG-Watch02B -> TG-Watch
- D3: value (none) -> BAS16XV2T1G
- moved D3 4.65 mm to (32.9, 27.8)
- moved C14 4.24 mm to (31.5, 18.6), turned to 0 degrees
- moved C15 1.35 mm to (31.0, 24.0)
- moved C9 1.35 mm to (32.0, 24.0)
- moved R9 1.27 mm to (33.2, 24.0)
- moved U8 1.25 mm to (32.5, 21.0)
- moved R14 0.65 mm to (27.4, 11.2)
- moved C2 0.35 mm to (27.2, 15.0)
- moved R13 0.15 mm to (27.5, 12.8)
- moved C4 0.05 mm to (27.5, 13.8)
- renumbered 04 to 04.1
Routing:
- net SYS_EN: track 13.8 -> 16.9 mm, vias 0 -> 2
- net RESET: track 53.9 -> 51.1 mm
- net VSORS: track 51.3 -> 48.7 mm
- net 3V3: track 118.3 -> 120.0 mm, vias 13 -> 14
- net VBUS: track 61.0 -> 61.7 mm
- net USBD+: track 5.78 -> 6.31 mm
- net GND: vias 331 -> 346
