File: ordered/TG-Watch02B-rev04.brd (EAGLE design)
At the start: 36.8 x 40.6 mm, 66 parts, among them IC3 W25Q128JVSIQ TR, J1 USB-C-CON-TG_MOD-2295018-2.0, J2 DISP_1.54_LCMTF15423A-C_LCD+C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, J3 CON-BAT-TG-MEZ_FEMALE, Q3 DMG2305, U2 MICROBUILDER_LSM6DSOX, U3 VREG-TPS63036, U4 FAN5331SX, U5 MCP73831/OT, U6 LC709203F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

Commit message: pre-order
Parts:
- D3: value BAS16XV2T1G -> (none)
Changed lines of the file:
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@@
 <setting verticaltext="up"/>
 </settings>
-<grid distance="0.25" unitdist="mm" unit="mm" style="lines" multiple="1" display="yes" altdistance="0.125" altunitdist="mm" altunit="mm"/>
+<grid distance="0.035" unitdist="mm" unit="mm" style="lines" multiple="1" display="yes" altdistance="0.125" altunitdist="mm" altunit="mm"/>
 <layers>
 <layer number="1" name="Top" color="4" fill="1" visible="yes" active="yes"/>
@@
 </element>
 <element name="U$3" library="0TG-Lib v01.5" package="SWD_POGO" value="CON_SWD_POGO" x="26" y="35.5" smashed="yes" rot="R270"/>
-<element name="D3" library="0TG-Lib v01.5" package="SOD-523" value="BAS16XV2T1G" x="34.75" y="23.5" smashed="yes" rot="R180">
+<element name="D3" library="0TG-Lib v01.5" package="SOD-523" value="" x="34.75" y="23.5" smashed="yes" rot="R180">
 <attribute name="NAME" x="35.566" y="24.084" size="0.75" layer="25" font="vector" ratio="20" rot="R270"/>
 <attribute name="VALUE" x="34.034" y="24.224" size="0.4064" layer="27" ratio="10" rot="R180"/>
