File: recalcitrant/TG-Watch02B-rev04-highpwr.brd (EAGLE design)
At the start: 36.8 x 40.6 mm, 62 parts, among them IC3 W25Q128JVSIQ TR, Q3 DMG2305, U10 MCU-ATTINY10, U2 BQ27441-G1, U4 FAN5331SX, U7 DISP_1.54_LCMTF15423A-C_LCD+C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, U8 UNDERVOLT-TPS3702CX3, U9 MCP73831/OT

Commit message: pre-order
Parts:
- removed ISP1: CON-ICSP/ISP-AVR-POGO, 0TG-Lib v01.5:2X3_POGO_AVR
- removed SJ1: (no value), 0TG-Lib v01.5:SOLDERJUMPER_2WAY_OPEN_0603
- removed U$13: CON_SWD_POGO_USB, 0TG-Lib v01.5:SWD_POGO_USB
- removed U10: MCU-ATTINY10, 0TG-Lib v01.5:SOT23-6
- added C19, C20: 10uf, 0TG-Lib v01.5:MICROBUILDER__0402_NODIMS
- added D3: (no value), 0TG-Lib v01.5:SOD-523
- added J2: DISP_1.54_LCMTF15423A-C_LCD+CAPTCH_ASSEMBLY_DUALSIDE, 0TG-Lib v01.5:TF-LCM15423A-C_DUALSIDE
- added L2: 1uH, FPV_Static-Lib_v1.1:NONSTANDARD_INDUCTOR_5
- added R13: 10k, 0TG-Lib v01.5:TG_0402
- added R16: 330k, 0TG-Lib v01.5:TG_0402
- added R3: 11k, 0TG-Lib v01.5:TG_0402
- added U6: LC709203F, microbuilder:WDFN8_3X4_0.65
- C2, C4: value 1uf -> 10uf
- D1: value MBR120 -> NSR05T40XV2
- D2: device microbuilder:SOD-523 -> microbuilder:SOD-323
- R1: value .01 ohm -> 10k
- R11: value 220K -> 220R
- R15: value 10k -> 59k
- R8: value 100k -> 2.7K
- U$3: value MICROBUILDER_LSM6DSOX -> CON_SWD_POGO; device lsm6dsox_ism330dhc:MICROBUILDER_LGA-14L -> 0TG-Lib v01.5:SWD_POGO
- U2: value BQ27441-G1 -> MICROBUILDER_LSM6DSOX; device battery-management-temp:PDSO-N12 -> lsm6dsox_ism330dhc:MICROBUILDER_LGA-14L
- U7: value DISP_1.54_LCMTF15423A-C_LCD+CAPTCH_ASSEMBLY_DUALSIDE -> TPS63036YFGR; device 0TG-Lib v01.5:TF-LCM15423A-C_DUALSIDE -> TPS63036YFGR:BGA8N40P4X2_181X107X62N
- moved U$3 36.5 mm to (25.8, 36.0)
- moved U7 32.5 mm to (32.0, 29.5), turned to 270 degrees
- moved U2 22.9 mm to (4.25, 6.50), turned to 270 degrees
- moved R1 18.6 mm to (26.6, 32.8), turned to 180 degrees
- moved C2 14.1 mm to (32.0, 26.5), turned to 90 degrees
- moved C14 13.2 mm to (30.2, 22.8), turned to 270 degrees
- moved C4 12.7 mm to (31.0, 26.5)
- moved R15 12.0 mm to (29.0, 25.8)
- moved C9 9.84 mm to (32.0, 22.8), turned to 90 degrees
- moved R2 5.00 mm to (22.2, 6.25), turned to 180 degrees
- moved R6 2.15 mm to (22.8, 8.50), turned to 270 degrees
- moved HEDR2 2.02 mm to (28.2, 30.2)
- moved C5 1.52 mm to (33.0, 26.5)
- moved R7 1.52 mm to (23.8, 9.50), turned to 270 degrees
- moved U1 1.00 mm to (23.5, 30.2)
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- renumbered 02 to 04, U$1 to J1, U$11 to J3, U9 to U5
Connections:
- net A0 renamed A0_SMC_RESET
- net D13_UNUSED renamed D13_RESERVED
- removed net 1.8V: C4.2, U2.5
- removed net D12_SMC_RESET: ISP1.5, MDBT1.24, R15.2, U10.6
- removed net D5_REQ_PWR_RST: MDBT1.25, U10.4
- removed net GPOUT: U2.12
- removed net N$6: SJ1.2, SW2.P$2
- removed net SYSON_TPICLK: ISP1.3, R9.1, SJ1.1, U10.3, U3.3, U8.1
- removed net TS: U2.10
- removed net VBAT_RAW: C2.2, J3.P$1, J3.P$2, J3.P$6, J3.P$7, R1.2, R6.2, U2.6, U2.8
- new net D12_BAT_INT: MDBT1.24, R13.2, U6.4
- new net D5_RESERVED: MDBT1.25
- new net L1: L2.1, U7.B1
- new net L2: L2.2, U7.C1
- new net SENSE: R15.2, R16.2, U7.D2
- new net SYS_EN: D3.K, R9.1, U3.3, U7.A2, U8.1
- new net TSENSE: R3.2, U6.6
- new net TSW: R3.1, U6.5
- net 3V3: now also C19.2, C2.2, C4.2, J2.FPC11, J2.FPC12, J2.MEZ5, R1.2, R13.1, R16.1, U$3.6, U2.12, U2.5, U2.8, U7.D1; no longer U$13.6, U$3.12, U$3.5, U$3.8, U7.FPC11, U7.FPC12, U7.MEZ5
- net 9.6V: now also D2.C; no longer D2.K
- net ACCEL_INT1: now also U2.4; no longer U$3.4
- net ACCEL_INT2: now also U2.9; no longer U$3.9
- net D+: no longer U$13.8
- net D-: no longer U$13.9
- net D17_CTP_INT: now also J2.MEZ9; no longer U7.MEZ9
- net D18_CTP_RESET: now also J2.MEZ6; no longer U7.MEZ6
- net D19_TFT_RESET: now also J2.FPC8; no longer U7.FPC8
- net D20_TFT_DC: now also J2.FPC6; no longer U7.FPC6
- net D22_TFT_CS: now also J2.FPC7; no longer U7.FPC7
- net GND: now also C19.1, C20.1, J2.FPC1, J2.FPC10, J2.FPC2, J2.MEZ1, J2.MEZ2, J2.MEZ3, R15.1, U$3.5, U2.1, U2.6, U2.7, U6.1, U6.2, U7.B2, U7.C2; no longer ISP1.6, U$13.1, U$13.5, U$3.6, U$3.7, U10.2, U2.3, U2.EP, U2.EP1, U2.EP2, U2.EP3, U2.EP4, U7.FPC1, U7.FPC10, U7.FPC2, U7.MEZ1, U7.MEZ2, U7.MEZ3
- net MOSI: now also J2.FPC4; no longer U7.FPC4
- net N$1: now also J2.FPC3; no longer U7.FPC3
- net RESET: now also D3.A, R1.1, SW2.P$2, U$3.7; no longer ISP1.1, SJ1.3, U$13.7, U10.1
- net SCK: now also J2.FPC5; no longer U7.FPC5
- net SCL: now also J2.MEZ7, U2.13, U6.8; no longer U$3.13, U2.2, U7.MEZ7
- net SDA: now also J2.MEZ8, U2.14, U6.7; no longer U$3.14, U2.1, U7.MEZ8
- net SWDCLK: now also U$3.4; no longer U$13.4
- net SWDIO: now also U$3.3; no longer U$13.3
- net SWO: now also U$3.2; no longer U$13.2
- net VBAT: now also J3.P$1, J3.P$2, J3.P$6, J3.P$7, R6.2, U6.3; no longer R1.1, U2.7
- net VLED: now also J2.FPC9; no longer U7.FPC9
- net VSORS: now also C20.2, U7.A1; no longer ISP1.2, R15.1, U10.5
Routing:
- net VSORS: track 122.7 -> 66.9 mm, vias 8 -> 11
- net VBAT_RAW: track 45.8 -> 0.00 mm, vias 6 -> 0
- net SYSON_TPICLK: track 39.3 -> 0.00 mm, vias 4 -> 0
- net D12_SMC_RESET: track 31.2 -> 0.00 mm, vias 2 -> 0
- net D12_BAT_INT: track 0.00 -> 26.1 mm, vias 0 -> 2
- net SWDCLK: track 5.23 -> 30.7 mm, vias 1 -> 2
- net SWDIO: track 3.31 -> 27.8 mm, vias 1 -> 2
- net D5_REQ_PWR_RST: track 22.2 -> 0.00 mm, vias 2 -> 0
- net SWO: track 7.76 -> 26.1 mm, vias 1 -> 2
- net D5_RESERVED: track 0.00 -> 11.6 mm, vias 0 -> 1
- net RESET: track 41.6 -> 52.6 mm, vias 2 -> 4
- net SYS_EN: track 0.00 -> 9.79 mm, vias 0 -> 3
- net D+: track 37.9 -> 29.1 mm, vias 1 -> 0
- net BAT_CHRG_SET: track 7.86 -> 1.88 mm, vias 2 -> 0
- net GND: track 196.8 -> 191.1 mm, vias 285 -> 326
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- added copper zone on layer 1, net 3V3
- added copper zone on layer 1, net L1
- added copper zone on layer 1, net L2
- added copper zone on layer 1, net VSORS
Other:
- board text added: "BAT1"
- board text added: "J2"
- board text added: "U1"
- board text added: "U4"
- board text added: "U9"
