File: recalcitrant/TG-Watch02B-rev04-highpwr.sch (EAGLE design)
At the start: 66 parts, among them IC3 W25Q128JVSIQ TR, J1 USB-C-CON-TG_MOD-2295018-2.0, J2 DISP_1.54_LCMTF15423A-C_LCD+C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, J3 CON-BAT-TG-MEZ_FEMALE, Q3 DMG2305, U2 MICROBUILDER_LSM6DSOX, U3 VREG-TPS63036, U4 FAN5331SX, U5 MCP73831/OT, U6 LC709203F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

Commit message: pre-order
Parts:
- removed SW1: (no value), 0TG-Lib v01.5:BUTTON-SPST_TACT_RA_NO_ALIGN
- added C20: 10uf, 0TG-Lib v01.5:C-US__0402_NOMASK
- added SW2: (no value), 0TG-Lib v01.5:SWITCH_PUSHBUTTONC&K_KSS
- D3: value BAS16XV2T1G -> (none)
- L2: value 1uH - HMLQ20161B-1R0MDR -> 1uH
- U3: value VREG-TPS63036 -> (none); device 0TG-Lib v01.5:VREG-TPS63036-3.3V-1A-SWITCHING_NOSILK -> 0TG-Lib v01.4:VREG_STD_MIN_SOT23-5
- U7: value (none) -> TPS63036YFGR; device 0TG-Lib v01.4:VREG_STD_MIN_SOT23-5 -> TPS63036YFGR:TPS63036YFGR
Connections:
- net 3V3: now also U3.OUT, U7.VOUT; no longer U3.VOUT, U7.OUT
- net GND: now also C20.1, SW2.P$1, U7.PS/SYNC; no longer SW1G$1.P, U3.PS/SYNC
- net L1: now also U7.L1; no longer U3.L1
- net L2: now also U7.L2; no longer U3.L2
- net RESET: now also SW2.P$2; no longer SW1G$1.S
- net SENSE: now also U7.FB; no longer U3.FB
- net VSORS: now also C20.2, U3.IN, U7.VIN; no longer U3.VIN, U7.IN
Other:
- moved on the sheet: C13, C15, C19, C2, C3, C4, C7, C8, D1, J3, L2, Q3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
