File: recalcitrant/TG-Watch02B-rev04-single-reg.sch (EAGLE design)
At the start: 66 parts, among them IC3 W25Q128JVSIQ TR, J1 USB-C-CON-TG_MOD-2295018-2.0, J2 DISP_1.54_LCMTF15423A-C_LCD+C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, J3 CON-BAT-TG-MEZ_FEMALE, Q3 DMG2305, U2 MICROBUILDER_LSM6DSOX, U3 VREG-TPS63036, U4 FAN5331SX, U5 MCP73831/OT, U6 LC709203F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

Commit message: pre-order
Parts:
- removed C19, C2, C4: 10uf, 0TG-Lib v01.5:C-US__0402_NOMASK
- removed L2: 1uH - HMLQ20161B-1R0MDR, FPV_Static-Lib_v1.1:INDUCTOR_1UHMEDIUM_CURRENT
- removed R15: 59k, 0TG-Lib v01.5:R_TG_0402
- removed R16: 330k, 0TG-Lib v01.5:R_TG_0402
- removed SW1: (no value), 0TG-Lib v01.5:BUTTON-SPST_TACT_RA_NO_ALIGN
- removed U7: (no value), 0TG-Lib v01.4:VREG_STD_MIN_SOT23-5
- added SW2: (no value), 0TG-Lib v01.5:SWITCH_PUSHBUTTONC&K_KSS
- D3: value BAS16XV2T1G -> (none)
- U3: value VREG-TPS63036 -> (none); device 0TG-Lib v01.5:VREG-TPS63036-3.3V-1A-SWITCHING_NOSILK -> 0TG-Lib v01.4:VREG_STD_MIN_SOT23-5
Connections:
- removed net L1: L2.1, U3.L1
- removed net L2: L2.2, U3.L2
- removed net SENSE: R15.2, R16.2, U3.FB
- net 3V3: now also U3.OUT; no longer C19.2, C2.2, C4.2, R16.1, U3.VOUT, U7.OUT
- net GND: now also SW2.P$1; no longer C19.1, C2.1, C4.1, R15.1, SW1G$1.P, U3.PS/SYNC, U7.GND
- net RESET: now also SW2.P$2; no longer SW1G$1.S
- net SYS_EN: no longer U7.EN
- net VSORS: now also U3.IN; no longer U3.VIN, U7.IN
Other:
- moved on the sheet: C13, C15, C3, C7, C8, D1, J3, Q3, R13, R2, R3, R8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
