File: reisions/TG-Watch02B-rev02.brd (EAGLE design)
At the start: 36.8 x 40.6 mm, 62 parts, among them IC3 W25Q128JVSIQ TR, Q3 DMG2305, U10 MCU-ATTINY10, U2 BQ27441-G1, U4 FAN5331SX, U7 DISP_1.54_LCMTF15423A-C_LCD+C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, U8 UNDERVOLT-TPS3702CX3, U9 MCP73831/OT

Commit message: pre-order
Parts:
- D1: value NSR05T40XV2 -> MBR120
- D2: device microbuilder:SOD-323 -> microbuilder:SOD-523
- R11: value 220R -> 220K
- R8: value 2.7K -> 100k
- moved L1 0.55 mm to (34.5, 6.25)
- moved D2 0.14 mm to (32.8, 5.75), turned to 180 degrees
- renumbered ACCEL1 to U$3, BAT1 to U$11
Connections:
- net 9.6V: now also D2.K; no longer D2.C
Routing:
- net SYSON_TPICLK: track 39.3 -> 44.0 mm
- net GND: track 196.0 -> 196.8 mm, vias 284 -> 285
- net 9.6V: track 12.9 -> 13.7 mm
Other:
- board text removed: "BAT1"
- board text removed: "U1"
- board text removed: "U10"
- board text removed: "U4"
- board text removed: "U7"
- board text removed: "U9"
