File: reisions/TG-Watch02B-rev03.brd (EAGLE design)
At the start: 36.8 x 40.6 mm, 66 parts, among them IC3 W25Q128JVSIQ TR, J1 USB-C-CON-TG_MOD-2295018-2.0, J2 DISP_1.54_LCMTF15423A-C_LCD+C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, J3 CON-BAT-TG-MEZ_FEMALE, Q3 DMG2305, U2 MICROBUILDER_LSM6DSOX, U3 VREG-TPS63036, U4 FAN5331SX, U5 MCP73831/OT, U6 LC709203F, U8 UNDERVOLT-TPS3702CX3

Commit message: pre-order
Parts:
- removed C19: 10uf, 0TG-Lib v01.5:MICROBUILDER__0402_NODIMS
- removed D3: BAS16XV2T1G, 0TG-Lib v01.5:SOD-523
- removed J2: DISP_1.54_LCMTF15423A-C_LCD+CAPTCH_ASSEMBLY_DUALSIDE, 0TG-Lib v01.5:TF-LCM15423A-C_DUALSIDE
- removed L2: 1uH - HMLQ20161B-1R0MDR, FPV_Static-Lib_v1.1:NONSTANDARD_INDUCTOR_5
- removed R13: 10k, 0TG-Lib v01.5:TG_0402
- removed R16: 330k, 0TG-Lib v01.5:TG_0402
- removed R3: 11k, 0TG-Lib v01.5:TG_0402
- removed SW1: (no value), 0TG-Lib v01.5:MICROBUILDER_SPST_TACTILE_RA_NO_ALIGN
- removed U$3: CON_SWD_POGO, 0TG-Lib v01.5:SWD_POGO
- removed U6: LC709203F, microbuilder:WDFN8_3X4_0.65
- added ACCEL1: MICROBUILDER_LSM6DSOX, lsm6dsox_ism330dhc:MICROBUILDER_LGA-14L
- added ISP1: CON-ICSP/ISP-AVR-POGO, 0TG-Lib v01.5:2X3_POGO_AVR
- added SJ1: (no value), 0TG-Lib v01.5:SOLDERJUMPER_2WAY_OPEN_0603
- added SW2: (no value), 0TG-Lib v01.5:BTN_CK_KSS
- added U$13: CON_SWD_POGO_USB, 0TG-Lib v01.5:SWD_POGO_USB
- added U10: MCU-ATTINY10, 0TG-Lib v01.5:SOT23-6
- C2, C4: value 10uf -> 1uf
- R1: value 10k -> .01 ohm
- R15: value 59k -> 10k
- U2: value MICROBUILDER_LSM6DSOX -> BQ27441-G1; device lsm6dsox_ism330dhc:MICROBUILDER_LGA-14L -> battery-management-temp:PDSO-N12
- U3: value VREG-TPS63036 -> (none); device 0TG-Lib v01.5:TPS63036YFGR_BGA8N40P4X2_NOSILK -> 0TG-Lib v01.4:SOT23-5
- U7: value (none) -> DISP_1.54_LCMTF15423A-C_LCD+CAPTCH_ASSEMBLY_DUALSIDE; device 0TG-Lib v01.4:SOT23-5 -> 0TG-Lib v01.5:TF-LCM15423A-C_DUALSIDE
- moved R15 25.2 mm to (23.8, 36.5), turned to 270 degrees
- moved U2 22.9 mm to (25.2, 15.8), turned to 180 degrees
- moved U7 21.5 mm to (18.4, 0.00), turned to 0 degrees
- moved R1 18.4 mm to (22.2, 14.8), turned to 270 degrees
- moved C14 13.3 mm to (23.8, 34.2), turned to 90 degrees
- moved C9 9.78 mm to (33.3, 32.5), turned to 180 degrees
- moved C4 6.24 mm to (22.2, 17.2), turned to 90 degrees
- moved R2 5.00 mm to (26.2, 9.25), turned to 270 degrees
- moved C5 4.76 mm to (32.8, 25.0), turned to 90 degrees
- moved R6 2.15 mm to (24.5, 9.75), turned to 0 degrees
- moved C2 1.82 mm to (28.0, 13.0), turned to 180 degrees
- moved R7 1.52 mm to (22.2, 9.75), turned to 0 degrees
- moved C11 1.46 mm to (26.8, 27.0)
- moved HEDR2 1.24 mm to (30.0, 29.2)
- moved C12 1.01 mm to (21.5, 32.8)
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- renumbered 04 to 02, J1 to U$1, J3 to BAT1, U5 to U9
Connections:
- net A0_SMC_RESET renamed A0
- net D13_RESERVED renamed D13_UNUSED
- removed net D12_BAT_INT: MDBT1.24, R13.2, U6.4
- removed net D5_RESERVED: MDBT1.25
- removed net L1: L2.1, U3.B1
- removed net L2: L2.2, U3.C1
- removed net SENSE: R15.2, R16.2, U3.D2
- removed net SYS_EN: D3.K, R9.1, U3.A2, U7.3, U8.1
- removed net TSENSE: R3.2, U6.6
- removed net TSW: R3.1, U6.5
- new net 1.8V: C4.2, U2.5
- new net D12_SMC_RESET: ISP1.5, MDBT1.24, R15.2, U10.6
- new net D5_REQ_PWR_RST: MDBT1.25, U10.4
- new net GPOUT: U2.12
- new net N$6: SJ1.2, SW2.P$2
- new net SYSON_TPICLK: ISP1.3, R9.1, SJ1.1, U10.3, U3.3, U8.1
- new net TS: U2.10
- new net VBAT_RAW: BAT1.P$1, BAT1.P$2, BAT1.P$6, BAT1.P$7, C2.2, R1.2, R6.2, U2.6, U2.8
- net 3V3: now also ACCEL1.12, ACCEL1.5, ACCEL1.8, U$13.6, U3.5, U7.FPC11, U7.FPC12, U7.MEZ5; no longer C19.2, C2.2, C4.2, J2.FPC11, J2.FPC12, J2.MEZ5, R1.2, R13.1, R16.1, U$3.6, U2.12, U2.5, U2.8, U3.D1, U7.5
- net ACCEL_INT1: now also ACCEL1.4; no longer U2.4
- net ACCEL_INT2: now also ACCEL1.9; no longer U2.9
- net D+: now also U$13.8
- net D-: now also U$13.9
- net D17_CTP_INT: now also U7.MEZ9; no longer J2.MEZ9
- net D18_CTP_RESET: now also U7.MEZ6; no longer J2.MEZ6
- net D19_TFT_RESET: now also U7.FPC8; no longer J2.FPC8
- net D20_TFT_DC: now also U7.FPC6; no longer J2.FPC6
- net D22_TFT_CS: now also U7.FPC7; no longer J2.FPC7
- net GND: now also ACCEL1.1, ACCEL1.6, ACCEL1.7, ISP1.6, SW2.P$1, U$13.1, U$13.5, U10.2, U2.3, U2.EP, U2.EP1, U2.EP2, U2.EP3, U2.EP4, U3.2, U7.FPC1, U7.FPC10, U7.FPC2, U7.MEZ1, U7.MEZ2, U7.MEZ3; no longer C19.1, J2.FPC1, J2.FPC10, J2.FPC2, J2.MEZ1, J2.MEZ2, J2.MEZ3, R15.1, SW1.1, U$3.1, U$3.5, U2.1, U2.6, U2.7, U3.B2, U3.C2, U6.1, U6.2, U7.2
- net MOSI: now also U7.FPC4; no longer J2.FPC4
- net N$1: now also U7.FPC3; no longer J2.FPC3
- net RESET: now also ISP1.1, SJ1.3, U$13.7, U10.1; no longer D3.A, R1.1, SW1.2, U$3.7
- net SCK: now also U7.FPC5; no longer J2.FPC5
- net SCL: now also ACCEL1.13, U2.2, U7.MEZ7; no longer J2.MEZ7, U2.13, U6.8
- net SDA: now also ACCEL1.14, U2.1, U7.MEZ8; no longer J2.MEZ8, U2.14, U6.7
- net SWDCLK: now also U$13.4; no longer U$3.4
- net SWDIO: now also U$13.3; no longer U$3.3
- net SWO: now also U$13.2; no longer U$3.2
- net VBAT: now also R1.1, U2.7; no longer BAT1.P$1, BAT1.P$2, BAT1.P$6, BAT1.P$7, R6.2, U6.3
- net VLED: now also U7.FPC9; no longer J2.FPC9
- net VSORS: now also ISP1.2, R15.1, U10.5, U3.1; no longer U3.A1, U7.1
Routing:
- net VSORS: track 51.3 -> 122.9 mm, vias 17 -> 8
- net 3V3: track 118.3 -> 166.8 mm, vias 13 -> 10
- net VBAT_RAW: track 0.00 -> 45.8 mm, vias 0 -> 6
- net SYSON_TPICLK: track 0.00 -> 39.3 mm, vias 0 -> 4
- net D12_SMC_RESET: track 0.00 -> 31.2 mm, vias 0 -> 2
- net SWDCLK: track 31.2 -> 5.23 mm, vias 2 -> 1
- net D12_BAT_INT: track 25.6 -> 0.00 mm, vias 2 -> 0
- net SWDIO: track 28.3 -> 3.31 mm, vias 2 -> 1
- net D5_REQ_PWR_RST: track 0.00 -> 22.2 mm, vias 0 -> 2
- net SWO: track 26.6 -> 7.76 mm, vias 2 -> 1
- net GND: track 177.8 -> 196.0 mm, vias 331 -> 284
- net SYS_EN: track 13.8 -> 0.00 mm
- net RESET: track 53.9 -> 41.6 mm, vias 4 -> 2
- net D5_RESERVED: track 11.6 -> 0.00 mm, vias 1 -> 0
- net D+: track 29.1 -> 37.9 mm, vias 0 -> 1
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- removed copper zone on layer 1, net 3V3
- removed copper zone on layer 1, net L1
- removed copper zone on layer 1, net L2
- removed copper zone on layer 1, net VSORS
- removed copper zone on layer 16, net VSORS
Other:
- board text added: "U10"
- board text added: "U7"
- board text removed: "J2"
